File: src/Qwiic-UART.kicad_sch (KiCad schematic)
At the start: 12 parts, among them J1 QWIIC, J2 QWIIC, J3 FTDI, U1 SC16IS740, X1 ECS-2520MVLC-018-BN-TR

Commit message: Made some refinements
Parts:
- removed JP1, JP2: SolderJumper_3_Open, Jumper:SolderJumper-3_P1.3mm_Open_RoundedPad1.0x1.5mm, symbol Jumper:SolderJumper_3_Open
- added JP1: SolderJumper_2_Bridged, Jumper:SolderJumper-2_P1.3mm_Bridged_RoundedPad1.0x1.5mm, symbol Jumper:SolderJumper_2_Bridged
- added JP2, JP3, JP4: SolderJumper_2_Open, Jumper:SolderJumper-2_P1.3mm_Open_RoundedPad1.0x1.5mm, symbol Jumper:SolderJumper_2_Open
- J1, J2: footprint Connector_JST:JST_SH_BM04B-SRSS-TB_1x04-1MP_P1.00mm_Vertical -> Connector_JST:JST_SH_SM04B-SRSS-TB_1x04-1MP_P1.00mm_Horizontal
- J3, J4: footprint Connector_PinHeader_2.54mm:PinHeader_1x06_P2.54mm_Vertical -> Project_Footprints:PinHeader_1x06_P2.54mm
Connections:
- net A1 is gone; now on net +3.3V: U1.3 (A1/SI)
- net +3.3V: now also J1.2 (Pin_2), J2.2 (Pin_2), JP1.1 (A); no longer J1.3 (Pin_3), J2.3 (Pin_3)
- net A0: now also JP1.2 (B), JP2.2 (B), JP3.2 (B), JP4.2 (B)
- net GND: now also J1.1 (Pin_1), J2.1 (Pin_1), JP2.1 (A); no longer J1.4 (Pin_4), J2.4 (Pin_4)
- net RX: now also J3.4 (Pin_4); no longer J3.5 (Pin_5)
- net SCL: now also J1.4 (Pin_4), J2.4 (Pin_4), JP3.1 (A); no longer J1.1 (Pin_1), J2.1 (Pin_1)
- net SDA: now also J1.3 (Pin_3), J2.3 (Pin_3), JP4.1 (A); no longer J1.2 (Pin_2), J2.2 (Pin_2)
- net TX: now also J3.5 (Pin_5); no longer J3.4 (Pin_4)
- net ~{CTS}: now also J3.6 (Pin_6); no longer J3.2 (Pin_2)
- net ~{RTS}: now also J3.2 (Pin_2); no longer J3.6 (Pin_6)
Other:
- moved on the sheet: J1, J2

Commit message: Added/generated essential files
Parts:
- J3, J4: now left out of the parts list
- U1: value SC16IS740 -> SC16IS741A
Other:
- note added: "Documentation and source files can be found at https://github.com/CMB27/Qwiic-UART."
- company: (none) -> Designer: C. M. Bulliner
- title: (none) -> Qwiic UART
- moved on the sheet: C1, C2, J2, J3, J4, R1, R2, U1, X1
